File: PCB_Keyboard.kicad_pcb (KiCad board)
At the start: 0 parts

Commit message: Add Type-C Submodule
Parts:
- added +/=1: MX-NoLED, MX_Only:MXOnly-1U, F.Cu at (254.0, 44.5)
- added -/_1: MX-NoLED, MX_Only:MXOnly-1U, F.Cu at (234.9, 44.5)
- added Backspace1: MX-NoLED, MX_Only:MXOnly-2U, F.Cu at (282.6, 44.5)
- added C1: 1uF, Capacitor_SMD:C_0805_2012Metric, F.Cu at (73.9, 173.3)
- added C2: 0.1uF, Capacitor_SMD:C_0805_2012Metric, F.Cu at (73.9, 176.3)
- added C3: 0.1uF, Capacitor_SMD:C_0805_2012Metric, F.Cu at (73.9, 179.3)
- added C4: 0.1uF, Capacitor_SMD:C_0805_2012Metric, F.Cu at (73.9, 182.3)
- added C5: 10uF, Capacitor_SMD:C_0805_2012Metric, F.Cu at (73.9, 185.3)
- added C6: 22pF, Capacitor_SMD:C_0805_2012Metric, F.Cu at (73.9, 188.3)
- added C7: 22pF, Capacitor_SMD:C_0805_2012Metric, F.Cu at (73.9, 191.3)
- added D1: D_Small, Diode_SMD:D_SOD-123, F.Cu at (299.3, 142.1)
- added D10: D_Small, Diode_SMD:D_SOD-123, F.Cu at (299.3, 172.2)
- added D11: D_Small, Diode_SMD:D_SOD-123, F.Cu at (299.3, 175.6)
- added D12: D_Small, Diode_SMD:D_SOD-123, F.Cu at (299.3, 178.9)
- added D13: D_Small, Diode_SMD:D_SOD-123, F.Cu at (305.1, 142.1)
- added D14: D_Small, Diode_SMD:D_SOD-123, F.Cu at (305.1, 145.4)
- added D15: D_Small, Diode_SMD:D_SOD-123, F.Cu at (305.1, 148.8)
- added D16: D_Small, Diode_SMD:D_SOD-123, F.Cu at (305.1, 152.1)
- added D17: D_Small, Diode_SMD:D_SOD-123, F.Cu at (305.1, 155.5)
- added D18: D_Small, Diode_SMD:D_SOD-123, F.Cu at (305.1, 158.8)
- added D19: D_Small, Diode_SMD:D_SOD-123, F.Cu at (305.1, 162.2)
- added D2: D_Small, Diode_SMD:D_SOD-123, F.Cu at (299.3, 145.4)
- added D20: D_Small, Diode_SMD:D_SOD-123, F.Cu at (305.1, 165.5)
- added D21: D_Small, Diode_SMD:D_SOD-123, F.Cu at (305.1, 168.9)
- added D22: D_Small, Diode_SMD:D_SOD-123, F.Cu at (305.1, 172.2)
- added D23: D_Small, Diode_SMD:D_SOD-123, F.Cu at (305.1, 175.6)
- added D24: D_Small, Diode_SMD:D_SOD-123, F.Cu at (305.1, 178.9)
- added D25: D_Small, Diode_SMD:D_SOD-123, F.Cu at (310.9, 142.1)
- added D26: D_Small, Diode_SMD:D_SOD-123, F.Cu at (310.9, 145.4)
- added D27: D_Small, Diode_SMD:D_SOD-123, F.Cu at (310.9, 148.8)
- added D28: D_Small, Diode_SMD:D_SOD-123, F.Cu at (310.9, 152.1)
- added D29: D_Small, Diode_SMD:D_SOD-123, F.Cu at (310.9, 155.5)
- added D3: D_Small, Diode_SMD:D_SOD-123, F.Cu at (299.3, 148.8)
- added D31: D_Small, Diode_SMD:D_SOD-123, F.Cu at (310.9, 158.8)
- added D32: D_Small, Diode_SMD:D_SOD-123, F.Cu at (310.9, 162.2)
- added D33: D_Small, Diode_SMD:D_SOD-123, F.Cu at (310.9, 165.5)
- added D34: D_Small, Diode_SMD:D_SOD-123, F.Cu at (310.9, 168.9)
- added D35: D_Small, Diode_SMD:D_SOD-123, F.Cu at (310.9, 172.2)
- added D37: D_Small, Diode_SMD:D_SOD-123, F.Cu at (310.9, 175.6)
- added D38: D_Small, Diode_SMD:D_SOD-123, F.Cu at (310.9, 178.9)
- added D39: D_Small, Diode_SMD:D_SOD-123, F.Cu at (316.7, 142.1)
- added D4: D_Small, Diode_SMD:D_SOD-123, F.Cu at (299.3, 152.1)
- added D40: D_Small, Diode_SMD:D_SOD-123, F.Cu at (316.7, 145.4)
- added D41: D_Small, Diode_SMD:D_SOD-123, F.Cu at (316.7, 148.8)
- added D42: D_Small, Diode_SMD:D_SOD-123, F.Cu at (316.7, 152.1)
- added D43: D_Small, Diode_SMD:D_SOD-123, F.Cu at (316.7, 155.5)
- added D44: D_Small, Diode_SMD:D_SOD-123, F.Cu at (316.7, 158.8)
- added D45: D_Small, Diode_SMD:D_SOD-123, F.Cu at (316.7, 162.2)
- added D46: D_Small, Diode_SMD:D_SOD-123, F.Cu at (316.7, 165.5)
- added D47: D_Small, Diode_SMD:D_SOD-123, F.Cu at (316.7, 168.9)
- added D48: D_Small, Diode_SMD:D_SOD-123, F.Cu at (316.7, 172.2)
- added D49: D_Small, Diode_SMD:D_SOD-123, F.Cu at (316.7, 175.6)
- added D5: D_Small, Diode_SMD:D_SOD-123, F.Cu at (299.3, 155.5)
- added D50: D_Small, Diode_SMD:D_SOD-123, F.Cu at (316.7, 178.9)
- added D51: D_Small, Diode_SMD:D_SOD-123, F.Cu at (322.5, 142.1)
- added D52: D_Small, Diode_SMD:D_SOD-123, F.Cu at (322.5, 145.4)
- added D53: D_Small, Diode_SMD:D_SOD-123, F.Cu at (322.5, 148.8)
- added D54: D_Small, Diode_SMD:D_SOD-123, F.Cu at (322.5, 152.1)
- added D55: D_Small, Diode_SMD:D_SOD-123, F.Cu at (322.5, 155.5)
- added D56: D_Small, Diode_SMD:D_SOD-123, F.Cu at (322.5, 158.8)
- added D57: D_Small, Diode_SMD:D_SOD-123, F.Cu at (322.5, 162.2)
- added D58: D_Small, Diode_SMD:D_SOD-123, F.Cu at (322.5, 165.5)
- added D6: D_Small, Diode_SMD:D_SOD-123, F.Cu at (299.3, 158.8)
- added D61: D_Small, Diode_SMD:D_SOD-123, F.Cu at (322.5, 168.9)
- added D62: D_Small, Diode_SMD:D_SOD-123, F.Cu at (322.5, 172.2)
- added D63: D_Small, Diode_SMD:D_SOD-123, F.Cu at (322.5, 175.6)
- added D64: D_Small, Diode_SMD:D_SOD-123, F.Cu at (322.5, 178.9)
- added D65: D_Small, Diode_SMD:D_SOD-123, F.Cu at (328.3, 142.1)
- added D66: D_Small, Diode_SMD:D_SOD-123, F.Cu at (328.3, 145.4)
- added D68: D_Small, Diode_SMD:D_SOD-123, F.Cu at (328.3, 148.8)
- added D69: D_Small, Diode_SMD:D_SOD-123, F.Cu at (328.3, 152.1)
- added D7: D_Small, Diode_SMD:D_SOD-123, F.Cu at (299.3, 162.2)
- added D70: D_Small, Diode_SMD:D_SOD-123, F.Cu at (328.3, 155.5)
- added D71: D_Small, Diode_SMD:D_SOD-123, F.Cu at (328.3, 158.8)
- added D73: D_Small, Diode_SMD:D_SOD-123, F.Cu at (328.3, 162.2)
- added D75: D_Small, Diode_SMD:D_SOD-123, F.Cu at (328.3, 165.5)
- added D77: D_Small, Diode_SMD:D_SOD-123, F.Cu at (328.3, 168.9)
- added D78: D_Small, Diode_SMD:D_SOD-123, F.Cu at (328.3, 172.2)
- added D79: D_Small, Diode_SMD:D_SOD-123, F.Cu at (328.3, 175.6)
- added D8: D_Small, Diode_SMD:D_SOD-123, F.Cu at (299.3, 165.5)
- added D81: D_Small, Diode_SMD:D_SOD-123, F.Cu at (328.3, 178.9)
- added D83: D_Small, Diode_SMD:D_SOD-123, F.Cu at (334.1, 142.1)
- added D85: D_Small, Diode_SMD:D_SOD-123, F.Cu at (334.1, 145.4)
- added D87: D_Small, Diode_SMD:D_SOD-123, F.Cu at (334.1, 148.8)
- added D88: D_Small, Diode_SMD:D_SOD-123, F.Cu at (334.1, 152.1)
- added D89: D_Small, Diode_SMD:D_SOD-123, F.Cu at (334.1, 155.5)
- added D9: D_Small, Diode_SMD:D_SOD-123, F.Cu at (299.3, 168.9)
- added D90: D_Small, Diode_SMD:D_SOD-123, F.Cu at (334.1, 158.8)
- added D92: D_Small, Diode_SMD:D_SOD-123, F.Cu at (334.1, 162.2)
- added D93: D_Small, Diode_SMD:D_SOD-123, F.Cu at (334.1, 165.5)
- added D94: D_Small, Diode_SMD:D_SOD-123, F.Cu at (334.1, 168.9)
- added D95: D_Small, Diode_SMD:D_SOD-123, F.Cu at (334.1, 172.2)
- added D96: D_Small, Diode_SMD:D_SOD-123, F.Cu at (334.1, 175.6)
- added Delete/Insert1: MX-NoLED, MX_Only:MXOnly-1U, F.Cu at (311.1, 25.4)
- added F13: 500mA, Fuse:Fuse_1206_3216Metric, F.Cu at (89.6, 194.2)
- added Home1: MX-NoLED, MX_Only:MXOnly-1U, F.Cu at (311.1, 44.5)
- added MX."1: MX-NoLED, MX_Only:MXOnly-1U, F.Cu at (249.2, 82.5)
- added MX.:1: MX-NoLED, MX_Only:MXOnly-1U, F.Cu at (230.2, 82.5)
- added MX.<1: MX-NoLED, MX_Only:MXOnly-1U, F.Cu at (203.2, 101.6)
- added MX.>1: MX-NoLED, MX_Only:MXOnly-1U, F.Cu at (222.2, 101.6)
- added MX.?: MX-NoLED, MX_Only:MXOnly-1U, F.Cu at (241.3, 101.6)
- added MX.A1: MX-NoLED, MX_Only:MXOnly-1U, F.Cu at (58.7, 82.5)
- added MX.B1: MX-NoLED, MX_Only:MXOnly-1U, F.Cu at (146.1, 101.6)
- added MX.C1: MX-NoLED, MX_Only:MXOnly-1U, F.Cu at (108.0, 101.6)
- added MX.CapsLock1: MX-NoLED, MX_Only:MXOnly-1.75U, F.Cu at (32.5, 82.5)
- added MX.Command1: MX-NoLED, MX_Only:MXOnly-1.25U, F.Cu at (75.4, 120.7)
- added MX.Command2: MX-NoLED, MX_Only:MXOnly-1U, F.Cu at (215.9, 120.7)
- added MX.Ctrl1: MX-NoLED, MX_Only:MXOnly-1.25U, F.Cu at (27.8, 120.7)
- added MX.Ctrl2: MX-NoLED, MX_Only:MXOnly-1U, F.Cu at (254.0, 120.7)
- added MX.D1: MX-NoLED, MX_Only:MXOnly-1U, F.Cu at (96.8, 82.5)
- added MX.E1: MX-NoLED, MX_Only:MXOnly-1U, F.Cu at (92.1, 63.5)
- added MX.End1: MX-NoLED, MX_Only:MXOnly-1U, F.Cu at (311.1, 101.6)
- added MX.Enter1: MX-NoLED, MX_Only:MXOnly-2.25U, F.Cu at (280.2, 82.5)
- added MX.F1: MX-NoLED, MX_Only:MXOnly-1U, F.Cu at (115.9, 82.5)
- added MX.Fn1: MX-NoLED, MX_Only:MXOnly-1U, F.Cu at (234.9, 120.7)
- added MX.G1: MX-NoLED, MX_Only:MXOnly-1U, F.Cu at (134.9, 82.5)
- added MX.H1: MX-NoLED, MX_Only:MXOnly-1U, F.Cu at (154.0, 82.5)
- added MX.I1: MX-NoLED, MX_Only:MXOnly-1U, F.Cu at (187.3, 63.5)
- added MX.J1: MX-NoLED, MX_Only:MXOnly-1U, F.Cu at (173.0, 82.5)
- added MX.K1: MX-NoLED, MX_Only:MXOnly-1U, F.Cu at (192.1, 82.5)
- added MX.L1: MX-NoLED, MX_Only:MXOnly-1U, B.Cu at (211.1, 82.5)
- added MX.M1: MX-NoLED, MX_Only:MXOnly-1U, F.Cu at (184.2, 101.6)
- added MX.N1: MX-NoLED, MX_Only:MXOnly-1U, F.Cu at (165.1, 101.6)
- added MX.O1: MX-NoLED, MX_Only:MXOnly-1U, F.Cu at (206.4, 63.5)
- added MX.Option1: MX-NoLED, MX_Only:MXOnly-1.25U, F.Cu at (51.6, 120.7)
- added MX.P1: MX-NoLED, MX_Only:MXOnly-1U, F.Cu at (225.4, 63.5)
- added MX.PageDown1: MX-NoLED, MX_Only:MXOnly-1U, F.Cu at (311.1, 82.5)
- added MX.Q1: MX-NoLED, MX_Only:MXOnly-1U, F.Cu at (54.0, 63.5)
- added MX.R1: MX-NoLED, MX_Only:MXOnly-1U, F.Cu at (111.1, 63.5)
- added MX.S1: MX-NoLED, MX_Only:MXOnly-1U, F.Cu at (77.8, 82.5)
- added MX.ShiftFull1: MX-NoLED, MX_Only:MXOnly-2.25U, F.Cu at (37.3, 101.6)
- added MX.ShiftHalf1: MX-NoLED, MX_Only:MXOnly-1.75U, F.Cu at (267.5, 101.6)
- added MX.T1: MX-NoLED, MX_Only:MXOnly-1U, F.Cu at (130.2, 63.5)
- added MX.TabFull1: MX-NoLED, MX_Only:MXOnly-1.5U, F.Cu at (30.2, 63.5)
- added MX.Tilda1: MX-NoLED, MX_Only:MXOnly-1U, F.Cu at (25.4, 44.5)
- added MX.U1: MX-NoLED, MX_Only:MXOnly-1U, F.Cu at (168.3, 63.5)
- added MX.V1: MX-NoLED, MX_Only:MXOnly-1U, F.Cu at (127.0, 101.6)
- added MX.W1: MX-NoLED, MX_Only:MXOnly-1U, F.Cu at (73.0, 63.5)
- added MX.X1: MX-NoLED, MX_Only:MXOnly-1U, F.Cu at (88.9, 101.6)
- added MX.Y1: MX-NoLED, MX_Only:MXOnly-1U, F.Cu at (149.2, 63.5)
- added MX.Z1: MX-NoLED, MX_Only:MXOnly-1U, F.Cu at (68.3, 101.6)
- added MX.backslash1: MX-NoLED, MX_Only:MXOnly-1U, F.Cu at (282.6, 63.5)
- added MX.down1: MX-NoLED, MX_Only:MXOnly-1U, F.Cu at (292.1, 120.7)
- added MX.right1: MX-NoLED, MX_Only:MXOnly-1U, F.Cu at (311.1, 120.7)
- added MX.up1: MX-NoLED, MX_Only:MXOnly-1U, F.Cu at (346.9, 71.4)
- added MX.{1: MX-NoLED, MX_Only:MXOnly-1U, F.Cu at (244.5, 63.5)
- added MX.}1: MX-NoLED, MX_Only:MXOnly-1U, F.Cu at (263.5, 63.5)
- added MXNum.1: MX-NoLED, MX_Only:MXOnly-1U, F.Cu at (44.5, 44.5)
- added MXNum.2: MX-NoLED, MX_Only:MXOnly-1U, F.Cu at (63.5, 44.5)
- added MXNum.3: MX-NoLED, MX_Only:MXOnly-1U, F.Cu at (82.5, 44.5)
- added MXNum.4: MX-NoLED, MX_Only:MXOnly-1U, F.Cu at (101.6, 44.5)
- added MXNum.5: MX-NoLED, MX_Only:MXOnly-1U, F.Cu at (120.7, 44.5)
- added MXNum.6: MX-NoLED, MX_Only:MXOnly-1U, F.Cu at (139.7, 44.5)
- added MXNum.7: MX-NoLED, MX_Only:MXOnly-1U, F.Cu at (158.8, 44.5)
- added MXNum.8: MX-NoLED, MX_Only:MXOnly-1U, F.Cu at (177.8, 44.5)
- added NmLck1: MX-NoLED, MX_Only:MXOnly-1U, F.Cu at (273.1, 25.4)
- added Num.0: MX-NoLED, MX_Only:MXOnly-1U, F.Cu at (215.9, 44.5)
- added Num.9: MX-NoLED, MX_Only:MXOnly-1U, F.Cu at (196.8, 44.5)
- added Pageup1: MX-NoLED, MX_Only:MXOnly-1U, F.Cu at (311.1, 63.5)
- added R1: 10k, Resistor_SMD:R_0805_2012Metric, F.Cu at (92.8, 173.3)
- added R2: 22, Resistor_SMD:R_0805_2012Metric, F.Cu at (92.8, 176.2)
- added R3: 22, Resistor_SMD:R_0805_2012Metric, F.Cu at (92.8, 179.2)
- added R4: 10k, Resistor_SMD:R_0805_2012Metric, F.Cu at (92.8, 182.1)
- added SW1: SW_Push, random-keyboard-parts:SKQG-1155865, F.Cu at (91.5, 189.4)
- added ScrLk1: MX-NoLED, MX_Only:MXOnly-1U, F.Cu at (292.1, 25.4)
- added Spacebar1: MX-NoLED, MX_Only:MXOnly-6.25U, F.Cu at (146.8, 120.7)
- added U1: ATmega32U4-A, Package_QFP:TQFP-44_10x10mm_P0.8mm, F.Cu at (83.3, 179.0)
- added USB1: Molex-0548190589, random-keyboard-parts:Molex-0548190589, F.Cu at (80.4, 191.2)
- added Y1: 16MHz, Crystal:Crystal_SMD_3225-4Pin_3.2x2.5mm, F.Cu at (95.0, 194.8)
- added esc1: MX-NoLED, MX_Only:MXOnly-1U, F.Cu at (25.4, 25.4)
- added f1: MX-NoLED, MX_Only:MXOnly-1U, F.Cu at (44.5, 25.4)
- added f10: MX-NoLED, MX_Only:MXOnly-1U, F.Cu at (215.9, 25.4)
- added f11: MX-NoLED, MX_Only:MXOnly-1U, F.Cu at (234.9, 25.4)
- added f12: MX-NoLED, MX_Only:MXOnly-1U, F.Cu at (254.0, 25.4)
- added f2: MX-NoLED, MX_Only:MXOnly-1U, F.Cu at (63.5, 25.4)
- added f3: MX-NoLED, MX_Only:MXOnly-1U, F.Cu at (82.5, 25.4)
- added f4: MX-NoLED, MX_Only:MXOnly-1U, F.Cu at (101.6, 25.4)
- added f5: MX-NoLED, MX_Only:MXOnly-1U, F.Cu at (120.7, 25.4)
- added f6: MX-NoLED, MX_Only:MXOnly-1U, F.Cu at (139.7, 25.4)
- added f7: MX-NoLED, MX_Only:MXOnly-1U, F.Cu at (158.8, 25.4)
- added f8: MX-NoLED, MX_Only:MXOnly-1U, F.Cu at (177.8, 25.4)
- added f9: MX-NoLED, MX_Only:MXOnly-1U, F.Cu at (196.8, 25.4)
Other:
- copper layers 0 -> 2
