File: matrix.sch.kicad_sch (KiCad schematic)
At the start: 166 parts

Commit message: Add Type-C Submodule
Parts:
- removed D94, D96: D_Small, symbol Device:D_Small
- removed MX.down1, MX.right1: MX-NoLED, symbol MX_Alps_Hybrid:MX-NoLED
- added D30, D36, D59: D_Small, Diode_SMD:D_SOD-123, symbol Device:D_Small
- added Down1, Left1, Right1: MX-NoLED, MX_Only:MXOnly-1U, symbol MX_Alps_Hybrid:MX-NoLED
- +/=1, -/_1, Delete/Insert1, Home1, MX."1, MX.1, MX.:1, MX.<1, MX.>1, MX.A1, MX.B1, MX.C1, MX.Command2, MX.Ctrl2, MX.D1, MX.E1, MX.End1, MX.F1, MX.Fn1, MX.G1, MX.H1, MX.J1, MX.K1, MX.L1, MX.M1, MX.N1, MX.PageDown1, MX.Q1, MX.R1, MX.S1, MX.T1, MX.Tilda1, MX.U1, MX.V1, MX.W1, MX.X1, MX.Y1, MX.Z1, MX.backslash1, MX.up1, MXNum.1, MXNum.2, MXNum.3, MXNum.4, MXNum.5, MXNum.6, MXNum.7, MXNum.8, NmLck1, Num.0, Num.9, Pageup1, ScrLk1, esc1, f1, f10, f11, f12, f2, f3, f4, f5, f6, f7, f8, f9: footprint (none) -> MX_Only:MXOnly-1U
- Backspace1: footprint (none) -> MX_Only:MXOnly-2U
- D1, D10, D11, D12, D13, D14, D15, D16, D17, D18, D19, D2, D20, D21, D22, D23, D24, D25, D26, D27, D28, D29, D3, D31, D32, D33, D34, D35, D37, D38, D39, D4, D40, D41, D42, D43, D44, D45, D46, D47, D48, D49, D5, D50, D51, D52, D53, D54, D55, D56, D57, D58, D6, D61, D62, D63, D64, D65, D66, D68, D69, D7, D70, D71, D73, D75, D77, D78, D79, D8, D81, D83, D85, D87, D88, D89, D9, D90, D92, D93, D95: footprint (none) -> Diode_SMD:D_SOD-123
- MX.CapsLock1, MX.ShiftHalf1: footprint (none) -> MX_Only:MXOnly-1.75U
- MX.Command1, MX.Ctrl1, MX.Option1: footprint (none) -> MX_Only:MXOnly-1.25U
- MX.Enter1, MX.ShiftFull1: footprint (none) -> MX_Only:MXOnly-2.25U
- MX.I1: renamed from MX.U2; footprint (none) -> MX_Only:MXOnly-1U
- MX.O1: renamed from MX.I1; footprint (none) -> MX_Only:MXOnly-1U
- MX.P1: renamed from MX.O1; footprint (none) -> MX_Only:MXOnly-1U
- MX.TabFull1: footprint (none) -> MX_Only:MXOnly-1.5U
- MX.{1: renamed from MX.P1; footprint (none) -> MX_Only:MXOnly-1U
- MX.}1: renamed from MX.{1; footprint (none) -> MX_Only:MXOnly-1U
- Spacebar1: footprint (none) -> MX_Only:MXOnly-6.25U
Connections:
- net col10: now also MX.Command2.1 (COL)
- net col11: now also MX.Fn1.1 (COL); no longer MX.Command2.1 (COL)
- net col12: now also MX.Ctrl2.1 (COL); no longer MX.Fn1.1 (COL)
- net col13: now also Left1.1 (COL); no longer MX.Ctrl2.1 (COL)
- net col14: no longer Backspace1.1 (COL), MX.Enter1.1 (COL), MX.backslash1.1 (COL), MX.up1.1 (COL), ScrLk1.1 (COL)
- net col15: now also Right1.1 (COL)
- net row5: now also D30.1 (K), D36.1 (K), D59.1 (K)
- new net: Backspace1.1 (COL), Down1.1 (COL), MX.Enter1.1 (COL), MX.backslash1.1 (COL), MX.up1.1 (COL), ScrLk1.1 (COL)
- new net: D36.2 (A), Down1.2 (ROW)
- new net: D30.2 (A), Left1.2 (ROW)
- new net: D59.2 (A), Right1.2 (ROW)
Other:
- moved on the sheet: D88, D90, D92, MX.Command2, MX.Ctrl2, MX.Fn1
